Commit message: update launch

File: urdf/bot.urdf.xacro (robot description, xacro)
@@ -2,6 +2,6 @@
 <robot name="slambot_description"
     xmlns:xacro="http://www.ros.org/wiki/xacro">
-    <xacro:include filename="$(find slambot_description)/urdf/materials.xacro" />
-    <xacro:include filename="$(find slambot_description)/urdf/bot.trans" />
+    <xacro:include filename="$(find slambot_cartographer)/urdf/materials.xacro" />
+    <!-- <xacro:include filename="$(find slambot_cartographer)/urdf/bot.trans" /> -->
     <xacro:macro name="gazebo_description" params="link color">
         <gazebo reference="${link}">
@@ -22,5 +22,5 @@
             <origin xyz="0 0 0" rpy="0 0 0"/>
             <geometry>
-                <mesh filename="package://slambot_description/meshes/base_link.stl" scale="0.001 0.001 0.001"/>
+                <mesh filename="package://slambot_cartographer/meshes/base_link.stl" scale="0.001 0.001 0.001"/>
             </geometry>
             <material name="opaque202209238"/>
@@ -29,5 +29,5 @@
             <origin xyz="0 0 0" rpy="0 0 0"/>
             <geometry>
-                <mesh filename="package://slambot_description/meshes/base_link.stl" scale="0.001 0.001 0.001"/>
+                <mesh filename="package://slambot_cartographer/meshes/base_link.stl" scale="0.001 0.001 0.001"/>
             </geometry>
         </collision>
@@ -43,5 +43,5 @@
             <origin xyz="0.061083 0.088085 -0.002998" rpy="0 0 0"/>
             <geometry>
-                <mesh filename="package://slambot_description/meshes/Top2BottomSupport_v1_1.stl" scale="0.001 0.001 0.001"/>
+                <mesh filename="package://slambot_cartographer/meshes/Top2BottomSupport_v1_1.stl" scale="0.001 0.001 0.001"/>
             </geometry>
             <material name="opaque202209238"/>
@@ -50,5 +50,5 @@
             <origin xyz="0.061083 0.088085 -0.002998" rpy="0 0 0"/>
             <geometry>
-                <mesh filename="package://slambot_description/meshes/Top2BottomSupport_v1_1.stl" scale="0.001 0.001 0.001"/>
+                <mesh filename="package://slambot_cartographer/meshes/Top2BottomSupport_v1_1.stl" scale="0.001 0.001 0.001"/>
             </geometry>
         </collision>
@@ -64,5 +64,5 @@
             <origin xyz="-0.088917 0.088085 -0.002998" rpy="0 0 0"/>
             <geometry>
-                <mesh filename="package://slambot_description/meshes/Top2BottomSupport_v1_2.stl" scale="0.001 0.001 0.001"/>
+                <mesh filename="package://slambot_cartographer/meshes/Top2BottomSupport_v1_2.stl" scale="0.001 0.001 0.001"/>
             </geometry>
             <material name="opaque202209238"/>
@@ -71,5 +71,5 @@
             <origin xyz="-0.088917 0.088085 -0.002998" rpy="0 0 0"/>
             <geometry>
-                <mesh filename="package://slambot_description/meshes/Top2BottomSupport_v1_2.stl" scale="0.001 0.001 0.001"/>
+                <mesh filename="package://slambot_cartographer/meshes/Top2BottomSupport_v1_2.stl" scale="0.001 0.001 0.001"/>
             </geometry>
         </collision>
@@ -85,5 +85,5 @@
             <origin xyz="-0.036417 -0.126915 -0.002998" rpy="0 0 0"/>
             <geometry>
-                <mesh filename="package://slambot_description/meshes/Top2BottomSupport_v1_3.stl" scale="0.001 0.001 0.001"/>
+                <mesh filename="package://slambot_cartographer/meshes/Top2BottomSupport_v1_3.stl" scale="0.001 0.001 0.001"/>
             </geometry>
             <material name="opaque202209238"/>
@@ -92,5 +92,5 @@
             <origin xyz="-0.036417 -0.126915 -0.002998" rpy="0 0 0"/>
             <geometry>
-                <mesh filename="package://slambot_description/meshes/Top2BottomSupport_v1_3.stl" scale="0.001 0.001 0.001"/>
+                <mesh filename="package://slambot_cartographer/meshes/Top2BottomSupport_v1_3.stl" scale="0.001 0.001 0.001"/>
             </geometry>
         </collision>
@@ -106,5 +106,5 @@
             <origin xyz="0.008583 -0.126915 -0.002998" rpy="0 0 0"/>
             <geometry>
-                <mesh filename="package://slambot_description/meshes/Top2BottomSupport_v1_4.stl" scale="0.001 0.001 0.001"/>
+                <mesh filename="package://slambot_cartographer/meshes/Top2BottomSupport_v1_4.stl" scale="0.001 0.001 0.001"/>
             </geometry>
             <material name="opaque202209238"/>
@@ -113,5 +113,5 @@
             <origin xyz="0.008583 -0.126915 -0.002998" rpy="0 0 0"/>
             <geometry>
-                <mesh filename="package://slambot_description/meshes/Top2BottomSupport_v1_4.stl" scale="0.001 0.001 0.001"/>
+                <mesh filename="package://slambot_cartographer/meshes/Top2BottomSupport_v1_4.stl" scale="0.001 0.001 0.001"/>
             </geometry>
         </collision>
@@ -127,5 +127,5 @@
             <origin xyz="-0.088917 0.088085 -0.053998" rpy="0 0 0"/>
             <geometry>
-                <mesh filename="package://slambot_description/meshes/Top_v1_1.stl" scale="0.001 0.001 0.001"/>
+                <mesh filename="package://slambot_cartographer/meshes/Top_v1_1.stl" scale="0.001 0.001 0.001"/>
             </geometry>
             <material name="opaque202209238"/>
@@ -134,5 +134,5 @@
             <origin xyz="-0.088917 0.088085 -0.053998" rpy="0 0 0"/>
             <geometry>
-                <mesh filename="package://slambot_description/meshes/Top_v1_1.stl" scale="0.001 0.001 0.001"/>
+                <mesh filename="package://slambot_cartographer/meshes/Top_v1_1.stl" scale="0.001 0.001 0.001"/>
             </geometry>
         </collision>
@@ -148,5 +148,5 @@
             <origin xyz="-0.033917 0.048085 -0.053998" rpy="0 0 0"/>
             <geometry>
-                <mesh filename="package://slambot_description/meshes/20V_Battery_Holder_v1_1.stl" scale="0.001 0.001 0.001"/>
+                <mesh filename="package://slambot_cartographer/meshes/20V_Battery_Holder_v1_1.stl" scale="0.001 0.001 0.001"/>
             </geometry>
             <material name="opaque202209238"/>
@@ -155,5 +155,5 @@
             <origin xyz="-0.033917 0.048085 -0.053998" rpy="0 0 0"/>
             <geometry>
-                <mesh filename="package://slambot_description/meshes/20V_Battery_Holder_v1_1.stl" scale="0.001 0.001 0.001"/>
+                <mesh filename="package://slambot_cartographer/meshes/20V_Battery_Holder_v1_1.stl" scale="0.001 0.001 0.001"/>
             </geometry>
         </collision>
@@ -169,5 +169,5 @@
             <origin xyz="0.053583 0.050085 0.003002" rpy="0 0 0"/>
             <geometry>
-                <mesh filename="package://slambot_description/meshes/Motor_Bracket_v1_1.stl" scale="0.001 0.001 0.001"/>
+                <mesh filename="package://slambot_cartographer/meshes/Motor_Bracket_v1_1.stl" scale="0.001 0.001 0.001"/>
             </geometry>
             <material name="opaque202209238"/>
@@ -176,5 +176,5 @@
             <origin xyz="0.053583 0.050085 0.003002" rpy="0 0 0"/>
             <geometry>
-                <mesh filename="package://slambot_description/meshes/Motor_Bracket_v1_1.stl" scale="0.001 0.001 0.001"/>
+                <mesh filename="package://slambot_cartographer/meshes/Motor_Bracket_v1_1.stl" scale="0.001 0.001 0.001"/>
             </geometry>
         </collision>
@@ -190,5 +190,5 @@
             <origin xyz="-0.095417 0.066085 0.003002" rpy="0 0 0"/>
             <geometry>
-                <mesh filename="package://slambot_description/meshes/Motor_Bracket_v1_2.stl" scale="0.001 0.001 0.001"/>
+                <mesh filename="package://slambot_cartographer/meshes/Motor_Bracket_v1_2.stl" scale="0.001 0.001 0.001"/>
             </geometry>
             <material name="opaque202209238"/>
@@ -197,5 +197,5 @@
             <origin xyz="-0.095417 0.066085 0.003002" rpy="0 0 0"/>
             <geometry>
-                <mesh filename="package://slambot_description/meshes/Motor_Bracket_v1_2.stl" scale="0.001 0.001 0.001"/>
+                <mesh filename="package://slambot_cartographer/meshes/Motor_Bracket_v1_2.stl" scale="0.001 0.001 0.001"/>
             </geometry>
         </collision>
@@ -211,5 +211,5 @@
             <origin xyz="-0.103117 0.058085 0.024002" rpy="0 0 0"/>
             <geometry>
-                <mesh filename="package://slambot_description/meshes/Motor_GM25-370_v1_1.stl" scale="0.001 0.001 0.001"/>
+                <mesh filename="package://slambot_cartographer/meshes/Motor_GM25-370_v1_1.stl" scale="0.001 0.001 0.001"/>
             </geometry>
             <material name="opaque202209238"/>
@@ -218,5 +218,5 @@
             <origin xyz="-0.103117 0.058085 0.024002" rpy="0 0 0"/>
             <geometry>
-                <mesh filename="package://slambot_description/meshes/Motor_GM25-370_v1_1.stl" scale="0.001 0.001 0.001"/>
+                <mesh filename="package://slambot_cartographer/meshes/Motor_GM25-370_v1_1.stl" scale="0.001 0.001 0.001"/>
             </geometry>
         </collision>
@@ -232,5 +232,5 @@
             <origin xyz="0.075283 0.058085 0.024002" rpy="0 0 0"/>
             <geometry>
-                <mesh filename="package://slambot_description/meshes/Motor_GM25-370_v1_2.stl" scale="0.001 0.001 0.001"/>
+                <mesh filename="package://slambot_cartographer/meshes/Motor_GM25-370_v1_2.stl" scale="0.001 0.001 0.001"/>
             </geometry>
             <material name="opaque202209238"/>
@@ -239,5 +239,5 @@
             <origin xyz="0.075283 0.058085 0.024002" rpy="0 0 0"/>
             <geometry>
-                <mesh filename="package://slambot_description/meshes/Motor_GM25-370_v1_2.stl" scale="0.001 0.001 0.001"/>
+                <mesh filename="package://slambot_cartographer/meshes/Motor_GM25-370_v1_2.stl" scale="0.001 0.001 0.001"/>
             </geometry>
         </collision>
@@ -253,5 +253,5 @@
             <origin xyz="-0.110367 0.058085 0.024002" rpy="0 0 0"/>
             <geometry>
-                <mesh filename="package://slambot_description/meshes/RC_coupling_v1_1.stl" scale="0.001 0.001 0.001"/>
+                <mesh filename="package://slambot_cartographer/meshes/RC_coupling_v1_1.stl" scale="0.001 0.001 0.001"/>
             </geometry>
             <material name="opaque202209238"/>
@@ -260,5 +260,5 @@
             <origin xyz="-0.110367 0.058085 0.024002" rpy="0 0 0"/>
             <geometry>
-                <mesh filename="package://slambot_description/meshes/RC_coupling_v1_1.stl" scale="0.001 0.001 0.001"/>
+                <mesh filename="package://slambot_cartographer/meshes/RC_coupling_v1_1.stl" scale="0.001 0.001 0.001"/>
             </geometry>
         </collision>
@@ -274,5 +274,5 @@
             <origin xyz="0.082533 0.058085 0.024002" rpy="0 0 0"/>
             <geometry>
-                <mesh filename="package://slambot_description/meshes/RC_coupling_v1_2.stl" scale="0.001 0.001 0.001"/>
+                <mesh filename="package://slambot_cartographer/meshes/RC_coupling_v1_2.stl" scale="0.001 0.001 0.001"/>
             </geometry>
             <material name="opaque202209238"/>
@@ -281,5 +281,5 @@
             <origin xyz="0.082533 0.058085 0.024002" rpy="0 0 0"/>
             <geometry>
-                <mesh filename="package://slambot_description/meshes/RC_coupling_v1_2.stl" scale="0.001 0.001 0.001"/>
+                <mesh filename="package://slambot_cartographer/meshes/RC_coupling_v1_2.stl" scale="0.001 0.001 0.001"/>
             </geometry>
         </collision>
@@ -295,5 +295,5 @@
             <origin xyz="0.100283 0.058085 0.024002" rpy="0 0 0"/>
             <geometry>
-                <mesh filename="package://slambot_description/meshes/85mm_Wheel_v1_1.stl" scale="0.001 0.001 0.001"/>
+                <mesh filename="package://slambot_cartographer/meshes/85mm_Wheel_v1_1.stl" scale="0.001 0.001 0.001"/>
             </geometry>
             <material name="opaque202209238"/>
@@ -302,5 +302,5 @@
             <origin xyz="0.100283 0.058085 0.024002" rpy="0 0 0"/>
             <geometry>
-                <mesh filename="package://slambot_description/meshes/85mm_Wheel_v1_1.stl" scale="0.001 0.001 0.001"/>
+                <mesh filename="package://slambot_cartographer/meshes/85mm_Wheel_v1_1.stl" scale="0.001 0.001 0.001"/>
             </geometry>
             <surface>
@@ -324,5 +324,5 @@
             <origin xyz="-0.128117 0.058085 0.024002" rpy="0 0 0"/>
             <geometry>
-                <mesh filename="package://slambot_description/meshes/85mm_Wheel_v1_2.stl" scale="0.001 0.001 0.001"/>
+                <mesh filename="package://slambot_cartographer/meshes/85mm_Wheel_v1_2.stl" scale="0.001 0.001 0.001"/>
             </geometry>
             <material name="opaque202209238"/>
@@ -331,5 +331,5 @@
             <origin xyz="-0.128117 0.058085 0.024002" rpy="0 0 0"/>
             <geometry>
-                <mesh filename="package://slambot_description/meshes/85mm_Wheel_v1_2.stl" scale="0.001 0.001 0.001"/>
+                <mesh filename="package://slambot_cartographer/meshes/85mm_Wheel_v1_2.stl" scale="0.001 0.001 0.001"/>
             </geometry>
             <surface>
@@ -353,5 +353,5 @@
             <origin xyz="-0.041917 -0.026915 -0.058998" rpy="0 0 0"/>
             <geometry>
-                <mesh filename="package://slambot_description/meshes/lidarBase_v2_1.stl" scale="0.001 0.001 0.001"/>
+                <mesh filename="package://slambot_cartographer/meshes/lidarBase_v2_1.stl" scale="0.001 0.001 0.001"/>
             </geometry>
             <material name="opaque202209238"/>
@@ -360,5 +360,5 @@
             <origin xyz="-0.041917 -0.026915 -0.058998" rpy="0 0 0"/>
             <geometry>
-                <mesh filename="package://slambot_description/meshes/lidarBase_v2_1.stl" scale="0.001 0.001 0.001"/>
+                <mesh filename="package://slambot_cartographer/meshes/lidarBase_v2_1.stl" scale="0.001 0.001 0.001"/>
             </geometry>
         </collision>
@@ -375,5 +375,5 @@
             <origin xyz="-0.081917 -0.072915 0.003002" rpy="0 0 0"/>
             <geometry>
-                <mesh filename="package://slambot_description/meshes/CastorWheel_Socks_v3_1.stl" scale="0.001 0.001 0.001"/>
+                <mesh filename="package://slambot_cartographer/meshes/CastorWheel_Socks_v3_1.stl" scale="0.001 0.001 0.001"/>
             </geometry>
             <material name="opaque202209238"/>
@@ -382,5 +382,5 @@
             <origin xyz="-0.081917 -0.072915 0.003002" rpy="0 0 0"/>
             <geometry>
-                <mesh filename="package://slambot_description/meshes/CastorWheel_Socks_v3_1.stl" scale="0.001 0.001 0.001"/>
+                <mesh filename="package://slambot_cartographer/meshes/CastorWheel_Socks_v3_1.stl" scale="0.001 0.001 0.001"/>
             </geometry>
         </collision>
@@ -397,5 +397,5 @@
             <origin xyz="0.054083 -0.072915 0.003002" rpy="0 0 0"/>
             <geometry>
-                <mesh filename="package://slambot_description/meshes/CastorWheel_Socks_v3_2.stl" scale="0.001 0.001 0.001"/>
+                <mesh filename="package://slambot_cartographer/meshes/CastorWheel_Socks_v3_2.stl" scale="0.001 0.001 0.001"/>
             </geometry>
             <material name="opaque202209238"/>
@@ -404,5 +404,5 @@
             <origin xyz="0.054083 -0.072915 0.003002" rpy="0 0 0"/>
             <geometry>
-                <mesh filename="package://slambot_description/meshes/CastorWheel_Socks_v3_2.stl" scale="0.001 0.001 0.001"/>
+                <mesh filename="package://slambot_cartographer/meshes/CastorWheel_Socks_v3_2.stl" scale="0.001 0.001 0.001"/>
             </geometry>
         </collision>
@@ -418,5 +418,5 @@
             <origin xyz="0.054083 -0.072915 0.028202" rpy="0 0 0"/>
             <geometry>
-                <mesh filename="package://slambot_description/meshes/Caster_40mm_Swivel_plate_v1_1.stl" scale="0.001 0.001 0.001"/>
+                <mesh filename="package://slambot_cartographer/meshes/Caster_40mm_Swivel_plate_v1_1.stl" scale="0.001 0.001 0.001"/>
             </geometry>
             <material name="opaque180180180"/>
@@ -425,5 +425,5 @@
             <origin xyz="0.054083 -0.072915 0.028202" rpy="0 0 0"/>
             <geometry>
-                <mesh filename="package://slambot_description/meshes/Caster_40mm_Swivel_plate_v1_1.stl" scale="0.001 0.001 0.001"/>
+                <mesh filename="package://slambot_cartographer/meshes/Caster_40mm_Swivel_plate_v1_1.stl" scale="0.001 0.001 0.001"/>
             </geometry>
         </collision>
@@ -439,5 +439,5 @@
             <origin xyz="-0.081917 -0.072915 0.028202" rpy="0 0 0"/>
             <geometry>
-                <mesh filename="package://slambot_description/meshes/Caster_40mm_Swivel_plate_v1_2.stl" scale="0.001 0.001 0.001"/>
+                <mesh filename="package://slambot_cartographer/meshes/Caster_40mm_Swivel_plate_v1_2.stl" scale="0.001 0.001 0.001"/>
             </geometry>
             <material name="opaque180180180"/>
@@ -446,5 +446,5 @@
             <origin xyz="-0.081917 -0.072915 0.028202" rpy="0 0 0"/>
             <geometry>
-                <mesh filename="package://slambot_description/meshes/Caster_40mm_Swivel_plate_v1_2.stl" scale="0.001 0.001 0.001"/>
+                <mesh filename="package://slambot_cartographer/meshes/Caster_40mm_Swivel_plate_v1_2.stl" scale="0.001 0.001 0.001"/>
             </geometry>
         </collision>
@@ -460,5 +460,5 @@
             <origin xyz="-0.066917 -0.084915 0.034502" rpy="0 0 0"/>
             <geometry>
-                <mesh filename="package://slambot_description/meshes/Caster_40mm_Wheel_support_v1_1.stl" scale="0.001 0.001 0.001"/>
+                <mesh filename="package://slambot_cartographer/meshes/Caster_40mm_Wheel_support_v1_1.stl" scale="0.001 0.001 0.001"/>
             </geometry>
             <material name="opaque180180180"/>
@@ -467,5 +467,5 @@
             <origin xyz="-0.066917 -0.084915 0.034502" rpy="0 0 0"/>
             <geometry>
-                <mesh filename="package://slambot_description/meshes/Caster_40mm_Wheel_support_v1_1.stl" scale="0.001 0.001 0.001"/>
+                <mesh filename="package://slambot_cartographer/meshes/Caster_40mm_Wheel_support_v1_1.stl" scale="0.001 0.001 0.001"/>
             </geometry>
         </collision>
@@ -481,5 +481,5 @@
             <origin xyz="0.039083 -0.084915 0.034502" rpy="0 0 0"/>
             <geometry>
-                <mesh filename="package://slambot_description/meshes/Caster_40mm_Wheel_support_v1_2.stl" scale="0.001 0.001 0.001"/>
+                <mesh filename="package://slambot_cartographer/meshes/Caster_40mm_Wheel_support_v1_2.stl" scale="0.001 0.001 0.001"/>
             </geometry>
             <material name="opaque180180180"/>
@@ -488,5 +488,5 @@
             <origin xyz="0.039083 -0.084915 0.034502" rpy="0 0 0"/>
             <geometry>
-                <mesh filename="package://slambot_description/meshes/Caster_40mm_Wheel_support_v1_2.stl" scale="0.001 0.001 0.001"/>
+                <mesh filename="package://slambot_cartographer/meshes/Caster_40mm_Wheel_support_v1_2.stl" scale="0.001 0.001 0.001"/>
             </geometry>
         </collision>
@@ -502,5 +502,5 @@
             <origin xyz="-0.058117 -0.069415 0.053302" rpy="0 0 0"/>
             <geometry>
-                <mesh filename="package://slambot_description/meshes/Caster_40mm_Wheel_30mm_v1_1.stl" scale="0.001 0.001 0.001"/>
+                <mesh filename="package://slambot_cartographer/meshes/Caster_40mm_Wheel_30mm_v1_1.stl" scale="0.001 0.001 0.001"/>
             </geometry>
             <material name="opaque255255255"/>
@@ -509,5 +509,5 @@
             <origin xyz="-0.058117 -0.069415 0.053302" rpy="0 0 0"/>
             <geometry>
-                <mesh filename="package://slambot_description/meshes/Caster_40mm_Wheel_30mm_v1_1.stl" scale="0.001 0.001 0.001"/>
+                <mesh filename="package://slambot_cartographer/meshes/Caster_40mm_Wheel_30mm_v1_1.stl" scale="0.001 0.001 0.001"/>
             </geometry>
         </collision>
@@ -523,5 +523,5 @@
             <origin xyz="0.047883 -0.069415 0.053302" rpy="0 0 0"/>
             <geometry>
-                <mesh filename="package://slambot_description/meshes/Caster_40mm_Wheel_30mm_v1_2.stl" scale="0.001 0.001 0.001"/>
+                <mesh filename="package://slambot_cartographer/meshes/Caster_40mm_Wheel_30mm_v1_2.stl" scale="0.001 0.001 0.001"/>
             </geometry>
             <material name="opaque255255255"/>
@@ -530,10 +530,10 @@
             <origin xyz="0.047883 -0.069415 0.053302" rpy="0 0 0"/>
             <geometry>
-                <mesh filename="package://slambot_description/meshes/Caster_40mm_Wheel_30mm_v1_2.stl" scale="0.001 0.001 0.001"/>
+                <mesh filename="package://slambot_cartographer/meshes/Caster_40mm_Wheel_30mm_v1_2.stl" scale="0.001 0.001 0.001"/>
             </geometry>
         </collision>
     </link>
     <!-- <xacro:gazebo_description link="Caster_40mm_Wheel_30mm_v1_2" color="Gazebo/White"/> -->
-    <link name="LidarTop_v1_1">
+    <link name="laser">
         <inertial>
             <origin xyz="-0.00023825807528363684 -0.00028540122623983005 0.013754821872220838" rpy="0 0 0"/>
@@ -544,5 +544,5 @@
             <origin xyz="-0.013917 -0.054915 -0.088598" rpy="0 0 0"/>
             <geometry>
-                <mesh filename="package://slambot_description/meshes/LidarTop_v1_1.stl" scale="0.001 0.001 0.001"/>
+                <mesh filename="package://slambot_cartographer/meshes/LidarTop_v1_1.stl" scale="0.001 0.001 0.001"/>
             </geometry>
             <material name="opaque202209238"/>
@@ -551,5 +551,5 @@
             <origin xyz="-0.013917 -0.054915 -0.088598" rpy="0 0 0"/>
             <geometry>
-                <mesh filename="package://slambot_description/meshes/LidarTop_v1_1.stl" scale="0.001 0.001 0.001"/>
+                <mesh filename="package://slambot_cartographer/meshes/LidarTop_v1_1.stl" scale="0.001 0.001 0.001"/>
             </geometry>
         </collision>
@@ -679,5 +679,5 @@
         <origin xyz="-0.028 0.028 0.0296" rpy="0 0 0"/>
         <parent link="lidarBase_v2_1"/>
-        <child link="LidarTop_v1_1"/>
+        <child link="laser"/>
     </joint>
 </robot>
